Commit message: mod reaching points to work with current version of marco planningf

File: model/robots/edinburgh_mods.xacro (robot description, xacro)
@@ -51,5 +51,5 @@
   </link>
   <joint name="l_hand_face_joint" type="fixed">
-    <origin rpy="3.14159265359 0 1.57079632679" xyz="0.08 0.0 -0.04"/>
+    <origin rpy="3.14159265359 0 1.57079632679" xyz="0.07 0.0 -0.08"/>
     <parent link="l_hand_force_torque"/>
     <child link="l_hand_face"/>
@@ -101,5 +101,5 @@
   </link>
   <joint name="r_hand_face_joint" type="fixed">
-    <origin rpy="0 0 -1.57079632679" xyz="0.08 0 0.04"/>
+    <origin rpy="0 0 -1.57079632679" xyz="0.07 0 0.08"/>
     <parent link="r_hand_force_torque"/>
     <child link="r_hand_face"/>

Commit message: updates to hands and mods

File: model/robots/edinburgh_mods.xacro (robot description, xacro)
@@ -1,8 +1,8 @@
 <robot xmlns:xacro="http://ros.org/wiki/xacro" name="valkyrie">
   <!-- drake feet mods-->
-  <frame link="LeftFoot"  name="l_foot_sole" rpy="0 0 0" xyz="0.0426  0.0017 -0.07645"/>
-  <frame link="RightFoot" name="r_foot_sole" rpy="0 0 0" xyz="0.0426 -0.0017 -0.07645"/>
-  <frame link="LeftFoot"  name="l_foot_toe"  rpy="0 0 0" xyz="0.1728  0.0017 -0.07645"/>
-  <frame link="RightFoot" name="r_foot_toe"  rpy="0 0 0" xyz="0.1728 -0.0017 -0.07645"/>
+  <frame link="leftFoot"  name="l_foot_sole" rpy="0 0 0" xyz="0.0426  0.0017 -0.07645"/>
+  <frame link="rightFoot" name="r_foot_sole" rpy="0 0 0" xyz="0.0426 -0.0017 -0.07645"/>
+  <frame link="leftFoot"  name="l_foot_toe"  rpy="0 0 0" xyz="0.1728  0.0017 -0.07645"/>
+  <frame link="rightFoot" name="r_foot_toe"  rpy="0 0 0" xyz="0.1728 -0.0017 -0.07645"/>
   <!-- end drake feet mods-->
   <!-- drake left hand frames-->
@@ -22,5 +22,5 @@
   <joint name="l_hand_force_torque_joint" type="fixed">
     <origin rpy="-1.57079632679 0 1.57079632679" xyz="0 0 0"/>
-    <parent link="LeftPalm"/>
+    <parent link="leftPalm"/>
     <child link="l_hand_force_torque"/>
   </joint>
@@ -72,5 +72,5 @@
   <joint name="r_hand_force_torque_joint" type="fixed">
     <origin rpy="-1.57079632679 0 -1.57079632679" xyz="0 0 0"/>
-    <parent link="RightPalm"/>
+    <parent link="rightPalm"/>
     <child link="r_hand_force_torque"/>
   </joint>
@@ -108,30 +108,30 @@
   <!-- drake collision free groups-->
   <collision_filter_group name="feet">
-    <member link="LeftFoot"/>
-    <member link="RightFoot"/>
+    <member link="leftFoot"/>
+    <member link="rightFoot"/>
     <ignored_collision_filter_group collision_filter_group="feet"/>
   </collision_filter_group>
   <collision_filter_group name="core">
-    <member link="Torso"/>
-    <member link="TorsoYawLink"/>
-    <member link="TorsoPitchLink"/>
-    <member link="Pelvis"/>
-    <member link="LowerNeckPitchLink"/>
-    <member link="NeckYawLink"/>
-    <member link="UpperNeckPitchLink"/>
+    <member link="torso"/>
+    <member link="torsoYawLink"/>
+    <member link="torsoPitchLink"/>
+    <member link="pelvis"/>
+    <member link="lowerNeckPitchLink"/>
+    <member link="neckYawLink"/>
+    <member link="upperNeckPitchLink"/>
     <member link="head"/>
     <ignored_collision_filter_group collision_filter_group="core"/>
   </collision_filter_group>
   <collision_filter_group name="ignore_core">
-    <member link="RightShoulderRollLink"/>
-    <member link="LeftShoulderRollLink"/>
-    <member link="RightShoulderPitchLink"/>
-    <member link="LeftShoulderPitchLink"/>
+    <member link="rightShoulderRollLink"/>
+    <member link="leftShoulderRollLink"/>
+    <member link="rightShoulderPitchLink"/>
+    <member link="leftShoulderPitchLink"/>
     <ignored_collision_filter_group collision_filter_group="core"/>
   </collision_filter_group>
   <collision_filter_group name="r_uleg">
-    <member link="RightHipYawLink"/>
-    <member link="RightHipRollLink"/>
-    <member link="RightHipPitchLink"/>
+    <member link="rightHipYawLink"/>
+    <member link="rightHipRollLink"/>
+    <member link="rightHipPitchLink"/>
     <ignored_collision_filter_group collision_filter_group="core"/>
     <ignored_collision_filter_group collision_filter_group="r_uleg"/>
@@ -139,7 +139,7 @@
   </collision_filter_group>
   <collision_filter_group name="l_uleg">
-    <member link="LeftHipYawLink"/>
-    <member link="LeftHipRollLink"/>
-    <member link="LeftHipPitchLink"/>
+    <member link="leftHipYawLink"/>
+    <member link="leftHipRollLink"/>
+    <member link="leftHipPitchLink"/>
     <ignored_collision_filter_group collision_filter_group="core"/>
     <ignored_collision_filter_group collision_filter_group="r_uleg"/>
@@ -147,35 +147,35 @@
   </collision_filter_group>
   <collision_filter_group name="r_leg">
-    <member link="RightKneePitchLink"/>
-    <member link="RightAnklePitchLink"/>
-    <member link="RightFoot"/>
+    <member link="rightKneePitchLink"/>
+    <member link="rightAnklePitchLink"/>
+    <member link="rightFoot"/>
     <ignored_collision_filter_group collision_filter_group="r_leg"/>
     <ignored_collision_filter_group collision_filter_group="r_uleg"/>
   </collision_filter_group>
   <collision_filter_group name="l_leg">
-    <member link="LeftKneePitchLink"/>
-    <member link="LeftAnklePitchLink"/>
-    <member link="LeftFoot"/>
+    <member link="leftKneePitchLink"/>
+    <member link="leftAnklePitchLink"/>
+    <member link="leftFoot"/>
     <ignored_collision_filter_group collision_filter_group="l_leg"/>
     <ignored_collision_filter_group collision_filter_group="l_uleg"/>
   </collision_filter_group>
   <collision_filter_group name="r_arm">
-    <member link="RightShoulderPitchLink"/>
-    <member link="RightShoulderRollLink"/>
-    <member link="RightShoulderYawLink"/>
-    <member link="RightElbowPitchLink"/>
-    <member link="RightForearmLink"/>
-    <member link="RightWristRollLink"/>
-    <member link="RightPalm"/>
+    <member link="rightShoulderPitchLink"/>
+    <member link="rightShoulderRollLink"/>
+    <member link="rightShoulderYawLink"/>
+    <member link="rightElbowPitchLink"/>
+    <member link="rightForearmLink"/>
+    <member link="rightWristRollLink"/>
+    <member link="rightPalm"/>
     <ignored_collision_filter_group collision_filter_group="r_arm"/>
   </collision_filter_group>
   <collision_filter_group name="l_arm">
-    <member link="LeftShoulderPitchLink"/>
-    <member link="LeftShoulderRollLink"/>
-    <member link="LeftShoulderYawLink"/>
-    <member link="LeftElbowPitchLink"/>
-    <member link="LeftForearmLink"/>
-    <member link="LeftWristRollLink"/>
-    <member link="LeftPalm"/>
+    <member link="leftShoulderPitchLink"/>
+    <member link="leftShoulderRollLink"/>
+    <member link="leftShoulderYawLink"/>
+    <member link="leftElbowPitchLink"/>
+    <member link="leftForearmLink"/>
+    <member link="leftWristRollLink"/>
+    <member link="leftPalm"/>
     <ignored_collision_filter_group collision_filter_group="l_arm"/>
   </collision_filter_group>

File: model/robots/valkyrie_hand_left.xacro (robot description, xacro)
@@ -1,9 +1,9 @@
 <robot xmlns:xacro="http://ros.org/wiki/xacro" name="valkyrie_hand_left">
-    <xacro:property name="mesh_root" value="package://val_description/meshes"/>
-    <xacro:property name="prefix" value="Left"/>
+    <xacro:property name="mesh_root" value="package://val_description/model/meshes"/>
+    <xacro:property name="prefix" value="left"/>
     <xacro:property name="reflect" value="1"/>
-    <xacro:property name="WristPitchLinkName" value="LeftPalm"/>
-    <xacro:include filename="$(find val_description)/robots/common/generic_models.xacro" />
-    <xacro:include filename="$(find val_description)/robots/valkyrie_A/xacro/common/common_bodies.xacro" />
+    <xacro:property name="WristPitchLinkName" value="leftPalm"/>
+    <xacro:include filename="$(find val_description)/model/robots/common/xacro/generic_models.xacro" />
+    <xacro:include filename="$(find val_description)/model/robots/common/xacro/common_bodies.xacro" />
     <link name="plane::xy::base">
       <inertial>
@@ -27,7 +27,7 @@
                     material="Gold"
                     collision_mesh="${mesh_root}/arms/palm_${prefix}.dae"/>
-    <xacro:make_thumb prefix="Left" reflect="1" thumb_root_link="LeftPalm"/>
-    <xacro:make_index_finger prefix="Left" reflect="1" index_finger_root_link="LeftPalm"/>
-    <xacro:make_middle_finger prefix="Left" reflect="1" middle_finger_root_link="LeftPalm"/>
-    <xacro:make_pinky_finger prefix="Left" reflect="1" pinky_finger_root_link="LeftPalm"/>
+    <xacro:make_thumb prefix="left" reflect="1" thumb_root_link="leftPalm"/>
+    <xacro:make_index_finger prefix="left" reflect="1" index_finger_root_link="leftPalm"/>
+    <xacro:make_middle_finger prefix="left" reflect="1" middle_finger_root_link="leftPalm"/>
+    <xacro:make_pinky_finger prefix="left" reflect="1" pinky_finger_root_link="leftPalm"/>
 </robot>

File: model/robots/valkyrie_hand_right.xacro (robot description, xacro)
@@ -1,9 +1,9 @@
 <robot xmlns:xacro="http://ros.org/wiki/xacro" name="valkyrie_hand_right">
-    <xacro:property name="mesh_root" value="package://val_description/meshes"/>
-    <xacro:property name="prefix" value="Right"/>
+    <xacro:property name="mesh_root" value="package://val_description/model/meshes"/>
+    <xacro:property name="prefix" value="right"/>
     <xacro:property name="reflect" value="-1"/>
-    <xacro:property name="WristPitchLinkName" value="RightPalm"/>
-    <xacro:include filename="$(find val_description)/robots/common/generic_models.xacro" />
-    <xacro:include filename="$(find val_description)/robots/valkyrie_A/xacro/common/common_bodies.xacro" />
+    <xacro:property name="WristPitchLinkName" value="rightPalm"/>
+    <xacro:include filename="$(find val_description)/model/robots/common/xacro/generic_models.xacro" />
+    <xacro:include filename="$(find val_description)/model/robots/common/xacro/common_bodies.xacro" />
     <link name="plane::xy::base">
       <inertial>
@@ -27,7 +27,7 @@
                     material="Gold"
                     collision_mesh="${mesh_root}/arms/palm_${prefix}.dae"/>
-    <xacro:make_thumb prefix="Right" reflect="-1" thumb_root_link="RightPalm"/>
-    <xacro:make_index_finger prefix="Right" reflect="-1" index_finger_root_link="RightPalm"/>
-    <xacro:make_middle_finger prefix="Right" reflect="-1" middle_finger_root_link="RightPalm"/>
-    <xacro:make_pinky_finger prefix="Right" reflect="-1" pinky_finger_root_link="RightPalm"/>
+    <xacro:make_thumb prefix="right" reflect="-1" thumb_root_link="rightPalm"/>
+    <xacro:make_index_finger prefix="right" reflect="-1" index_finger_root_link="rightPalm"/>
+    <xacro:make_middle_finger prefix="right" reflect="-1" middle_finger_root_link="rightPalm"/>
+    <xacro:make_pinky_finger prefix="right" reflect="-1" pinky_finger_root_link="rightPalm"/>
 </robot>
